File: PowerSupply.kicad_sch (KiCad schematic)
At the start: 6 parts, among them J5 DC Barrel Jack, U4 AP62250smol

Commit message: Rev C, I think
Parts:
- removed TP1: TestPoint, TestPoint:TestPoint_Loop_D2.50mm_Drill1.0mm_LowProfile, symbol Connector:TestPoint
Changed lines of the file:
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@@
   (junction (at 44.45 35.56) (diameter 0) (color 0 0 0 0)
-  )
-  (junction (at 113.03 35.56) (diameter 0) (color 0 0 0 0)
   )
   (junction (at 64.77 35.56) (diameter 0) (color 0 0 0 0)
@@
     (pin "3")
   )
-  (symbol (lib_id "Connector:TestPoint") (at 113.03 35.56 270) (unit 1)
-    (in_bom yes) (on_board yes) (fields_autoplaced)
-    (property "Reference" "TP1" (id 0) (at 116.332 38.3445 90))
-    (property "Value" "TestPoint" (id 1) (at 116.332 41.1196 90))
-    (property "Footprint" "TestPoint:TestPoint_Loop_D2.50mm_Drill1.0mm_LowProfile" (id 2) (at 113.03 40.64 0)
-      (effects (font (size 1.27 1.27)) hide)
-    )
-    (property "Datasheet" "~" (id 3) (at 113.03 40.64 0)
-      (effects (font (size 1.27 1.27)) hide)
-    )
-    (pin "1")
-  )
 )
