File: smolDuino.kicad_pcb (KiCad board)
At the start: 2 copper layers, 68.6 x 53.3 mm, 71 parts, among them J1 USB_C_Receptacle_USB2.0, J2 2x3 SPI Header, J3 2x5 HV Outputs, J4 I^{2}C Connector, J5 DC Barrel Jack, J6 Battery Connector, P1 CONN_01X01, P2 CONN_01X01, P3 CONN_01X01, P4 CONN_01X01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

Commit message: Remove Gas Gauge IC
Parts:
- removed C9: 1uF, Capacitor_SMD:C_0603_1608Metric
- removed U7: LC709203FXE-05MH, MikeFootprintLib:WLCSP9-1.60x1.76mm
- MISC1, MISC2: value C -> D
Routing:
- net /IO19: track 83.3 -> 61.2 mm, vias 4 -> 2
- net /IO18: track 78.2 -> 59.9 mm, vias 4 -> 2
- net +BATT: track 15.4 -> 0.00 mm
- net GND: track 77.2 -> 73.3 mm, vias 286 -> 282
